Commit message: updated lens 'x' position

File: traxxas_robot_description/urdf/zed2.xacro (robot description, xacro)
@@ -70,5 +70,5 @@
         <parent link="zed2_camera_link" />
         <child link="zed2_left_lens_link" />
-        <origin xyz="${zed_length/2} ${(zed_width/2) - lens_radius - lens_offset} 0" rpy="0 0 0" />
+        <origin xyz="${zed_length/2 + 0.001} ${(zed_width/2) - lens_radius - lens_offset} 0" rpy="0 0 0" />
         <axis xyz="0 1 0" />
     </joint>
@@ -76,5 +76,5 @@
         <parent link="zed2_camera_link" />
         <child link="zed2_right_lens_link" />
-        <origin xyz="${zed_length/2} -${(zed_width/2) - lens_radius - lens_offset} 0" rpy="0 0 0" />
+        <origin xyz="${zed_length/2 + 0.001} -${(zed_width/2) - lens_radius - lens_offset} 0" rpy="0 0 0" />
         <axis xyz="0 1 0" />
     </joint>
