Commit message: Add Custom ZED2
ENG
- Implement ZED2 camera URDF Xacro model with right and left lens modules
- Configure stereo camera sensors in Gazebo with Gaussian noise simulation
- Add Gazebo plugins for image capture (640x480 resolution at 30 FPS)
- Integrate ROS-Gazebo bridges for image and camera_info topics
- Define optical frames with correct transformations for vision processing
- Update main URDF file to include ZED2 camera model
- Configure camera visualization in RViz with image display plugins
- Set noise parameters and capture range (0.1m - 15m)

ESP
- Implementar modelo URDF Xacro de cámara ZED2 con lentes derecho e izquierdo
- Configurar sensores de cámara estéreo en Gazebo con ruido gaussiano
- Añadir plugins de Gazebo para captura de imágenes (640x480, 30 FPS)
- Integrar puentes ROS-Gazebo para tópicos de imagen y información de cámara
- Definir frames ópticos con transformaciones correctas para procesamiento de visión
- Actualizar archivo URDF principal para incluir modelo ZED2
- Configurar visualización de cámaras en RViz con displays de imagen
- Establecer parámetros de ruido y rango de captura (0.1m - 15m)

File: traxxas_robot_description/urdf/common_properties.xacro (robot description, xacro)
@@ -15,4 +15,7 @@
     <material name="grey_dark">
         <color rgba="0.188 0.176 0.176 1.0"/>
+    </material>
+    <material name="zed_gray">
+        <color rgba="0.189 0.188 0.197 1.0"/>
     </material>
     <xacro:macro name="box_inertia" params="m l w h o_xyz o_rpy">

File: traxxas_robot_description/urdf/traxxas.urdf.xacro (robot description, xacro)
@@ -4,3 +4,6 @@
     <xacro:include filename="$(find traxxas_robot_description)/urdf/mobile_base.xacro" />
     <xacro:include filename="$(find traxxas_robot_description)/urdf/mobile_base_gazebo.xacro" />
+    <!-- The original design does not include any camera nor lidar.
+    To edit original design, comment the following lines.  -->
+    <xacro:include filename="$(find traxxas_robot_description)/urdf/zed2.xacro" />
 </robot>

Commit message: Add Custom Lane follower Camera
ENG
- Create new camera_lane.xacro file with lane follower camera model
- Include new camera in robot main assembly (traxxas.urdf.xacro)
- Configure camera geometry, inertial properties and Gazebo sensors for lane follower
- Add Gazebo-ROS bridge topics for lane follower camera image and camera_info streams
- Add lane follower camera visualization to RViz configuration
- Add camera links (base, pose, lens, optical) to RViz display configuration
- Include "white" material in common properties for camera base

ESP
- Nuevo archivo camera_lane.xacro con modelo de cámara para seguimiento de carriles
Incluir nueva cámara en el ensamblaje principal del robot (traxxas.urdf.xacro)
- Configuración de geometría, inercial y sensores de la cámara lane follower en Gazebo
- Añadidos tópicos de puente Gazebo-ROS para imagen y cámara_info de la cámara lane follower
- Agregada visualización de cámara lane follower en configuración de RViz
- Añadidos enlaces de la cámara (base, pose, lens, optical) a la configuración de RViz
- Incluido material "white" (blanco) en propiedades comunes para la base de la cámara

File: traxxas_robot_description/urdf/common_properties.xacro (robot description, xacro)
@@ -1,4 +1,7 @@
 <?xml version="1.0"?>
 <robot xmlns:xacro="http://www.ros.org/wiki/xacro">
+    <material name="white">
+        <color rgba="1 1 1 1" />
+    </material>
     <material name="blue">
         <color rgba="0 0 0.5 1" />

File: traxxas_robot_description/urdf/traxxas.urdf.xacro (robot description, xacro)
@@ -7,3 +7,4 @@
     To edit original design, comment the following lines.  -->
     <xacro:include filename="$(find traxxas_robot_description)/urdf/zed2.xacro" />
+    <xacro:include filename="$(find traxxas_robot_description)/urdf/camera_lane.xacro" />
 </robot>
