Commit message: Traxxas v2
ENG
- Configured Custom ZED 2 camera position to be positioned higher.
- Created base stand for the ZED 2 camera to position int higher and more chassis-centered in x axis.
- Removed secondary camera intended for line following.
- Modifications made to optimize sensor usage and for line-following tests using the ZED 2 camera.

ESP
- Se configuró la posición personalizada de la cámara ZED 2 para colocarla a mayor altura.
- Se creó una base (stand) para la cámara ZED 2 con el fin de elevarla y centrarla mejor respecto al chasis en el eje x.
- Se eliminó la cámara secundaria destinada al seguimiento de línea.
- Se realizaron modificaciones para optimizar el uso de sensores y las pruebas de seguimiento de línea utilizando la cámara ZED 2.

File: traxxas_robot_description/urdf/traxxas.urdf.xacro (robot description, xacro)
@@ -4,8 +4,8 @@
     <xacro:include filename="$(find traxxas_robot_description)/urdf/mobile_base.xacro" />
     <xacro:include filename="$(find traxxas_robot_description)/urdf/mobile_base_gazebo.xacro" />
-    <!-- The original design does not include any camera nor lidar.
+    <!-- The original design does not include any camera nor LiDAR.
     To edit original design, comment the following lines.  -->
     <xacro:include filename="$(find traxxas_robot_description)/urdf/zed2.xacro" />
-    <xacro:include filename="$(find traxxas_robot_description)/urdf/camera_lane.xacro" />
+    <!-- <xacro:include filename="$(find traxxas_robot_description)/urdf/camera_lane.xacro" /> -->
     <xacro:include filename="$(find traxxas_robot_description)/urdf/lidar.xacro" />
 </robot>

File: traxxas_robot_description/urdf/zed2.xacro (robot description, xacro)
@@ -7,6 +7,10 @@
     <xacro:property name="lens_radius" value="0.0095" />
     <xacro:property name="lens_offset" value="0.017" />
-    <xacro:property name="zed_length_position" value="0.053" />
+    <xacro:property name="zed_length_position" value="0.05353" />
     <xacro:property name="zed_mass" value="0.124" />
+    <!-- Stand properties -->
+    <xacro:property name="stand_length" value="${zed_length}" />
+    <xacro:property name="stand_width" value="0.072" />
+    <xacro:property name="stand_height" value="0.0214" />
     <!-- Functions -->
     <xacro:macro name="lens" params="prefix">
@@ -29,4 +33,20 @@
     </xacro:macro>
     <!-- Links -->
+    <link name="stand_link">
+        <xacro:box_inertia m="0.3" l="${stand_length}" w="${stand_width}" h="${stand_height}" o_xyz="0.0 0.0 ${stand_height/2}" o_rpy="0.0 0.0 0.0" />
+        <visual>
+            <origin xyz="0 0 0" rpy="0 0 0" />
+            <geometry>
+                <box size="${stand_length} ${stand_width} ${stand_height}" />
+            </geometry>
+            <material name="white" />
+        </visual>
+        <collision>
+            <origin xyz="0 0 0" rpy="0 0 0" />
+            <geometry>
+                <box size="${stand_length} ${stand_width} ${stand_height}" />
+            </geometry>
+        </collision>
+    </link>
     <link name="zed2_camera_link">
         <xacro:box_inertia l="${zed_length}" w="${zed_width}" h="${zed_height}"
@@ -61,8 +81,20 @@
         <origin xyz="0 0 0" rpy="${-pi/2} 0 ${-pi/2}"/>
     </joint>
-    <joint name="chassis_to_zed2_joint" type="fixed">
+    <!-- <joint name="chassis_to_zed2_joint" type="fixed">
         <parent link="chassis_link" />
         <child link="zed2_camera_link" />
         <origin xyz="${((chassis_length + zed_length)/2) - zed_length_position} 0 ${chassis_height + zed_height/2}" rpy="0 0 0" />
+        <axis xyz="0 1 0" />
+    </joint> -->
+    <joint name="chassis_to_stand" type="fixed">
+        <parent link="chassis_link" />
+        <child link="stand_link" />
+        <origin xyz="${(chassis_length/2) - (stand_length/2) - zed_length_position} 0 ${chassis_height + stand_height/2}" rpy="0 0 0" />
+        <axis xyz="1 0 0" />
+    </joint>
+    <joint name="stand_to_zed2" type="fixed">
+        <parent link="stand_link" />
+        <child link="zed2_camera_link" />
+        <origin xyz="0 0 ${stand_height/2 + zed_height/2}" rpy="0 0 0" />
         <axis xyz="0 1 0" />
     </joint>
