Commit message: Corrected Mobile Base
ENG
- Corrected invalid parameter values

ESP
- Corregidos parámetros con valores inválidos

File: traxxas_robot_description/urdf/mobile_base.xacro (robot description, xacro)
@@ -6,15 +6,15 @@
     <xacro:property name="chassis_width" value="0.18" />
     <xacro:property name="chassis_height" value="0.062" />
-    <xacro:property name="chassis_mass" value="7850*${chassis_length * chassis_width * chassis_height}" />
+    <xacro:property name="chassis_mass" value="${7850.0 * chassis_length * chassis_width * chassis_height}" />
     <!-- Front suspension dimensions -->
     <xacro:property name="front_suspension_length" value="0.03" />
     <xacro:property name="front_suspension_width" value="0.1" />
     <xacro:property name="front_suspension_height" value="0.09" />
-    <xacro:property name="front_suspension_mass" value="7850.0*${front_suspension_length * front_suspension_width * front_suspension_height}" />
+    <xacro:property name="front_suspension_mass" value="${7850.0 * front_suspension_length * front_suspension_width * front_suspension_height}" />
     <!--Rear suspension dimensions -->
     <xacro:property name="rear_suspension_length" value="0.05" />
     <xacro:property name="rear_suspension_width" value="0.11" />
     <xacro:property name="rear_suspension_height" value="0.105" />
-    <xacro:property name="rear_suspension_mass" value="7850.0*${rear_suspension_length * rear_suspension_width * rear_suspension_height}" />
+    <xacro:property name="rear_suspension_mass" value="${7850.0 * rear_suspension_length * rear_suspension_width * rear_suspension_height}" />
     <!-- Wheel dimensions -->
     <xacro:property name="wheel_radius" value="0.0535" />

Commit message: UPDATE steering
ENG
- Update in steering angles.

ESP
- Actualizado el ángulo de giro del volante.

File: traxxas_robot_description/urdf/mobile_base.xacro (robot description, xacro)
@@ -26,4 +26,5 @@
     <!-- Steering params -->
     <xacro:property name="max_steering_angle" value="0.5236" />
+    <xacro:property name="counter_max_steering_angle" value="0.349066" />
     <xacro:property name="max_steering_angular_vel" value="1.570796" />
     <xacro:property name="max_steering_effort" value="1.0" />
@@ -216,5 +217,5 @@
         <origin xyz="0 ${-(front_wheel_axis_width/2)} 0" rpy="0 0 0" />
         <axis xyz="0 0 1" />
-        <limit lower="${-max_steering_angle}" upper="${max_steering_angle}" effort="${max_steering_effort}" velocity="${max_steering_angular_vel}" />
+        <limit lower="${-max_steering_angle}" upper="${counter_max_steering_angle}" effort="${max_steering_effort}" velocity="${max_steering_angular_vel}" />
         <dynamics damping="0.1" friction="0.1"/>
     </joint>
@@ -232,5 +233,5 @@
         <origin xyz="0 ${(front_wheel_axis_width/2)} 0" rpy="0 0 0" />
         <axis xyz="0 0 1" />
-        <limit lower="${-max_steering_angle}" upper="${max_steering_angle}" effort="${max_steering_effort}" velocity="${max_steering_angular_vel}" />
+        <limit lower="${-counter_max_steering_angle}" upper="${max_steering_angle}" effort="${max_steering_effort}" velocity="${max_steering_angular_vel}" />
         <dynamics damping="0.1" friction="0.1"/>
     </joint>

Commit message: Update robot description - Updated chassis height - Updated camera image resolution - Updated rviz configuration

File: traxxas_robot_description/urdf/mobile_base.xacro (robot description, xacro)
@@ -5,15 +5,15 @@
     <xacro:property name="chassis_length" value="0.31" />
     <xacro:property name="chassis_width" value="0.18" />
-    <xacro:property name="chassis_height" value="0.062" />
+    <xacro:property name="chassis_height" value="0.07869" />
     <xacro:property name="chassis_mass" value="${7850.0 * chassis_length * chassis_width * chassis_height}" />
     <!-- Front suspension dimensions -->
     <xacro:property name="front_suspension_length" value="0.03" />
     <xacro:property name="front_suspension_width" value="0.1" />
-    <xacro:property name="front_suspension_height" value="0.09" />
+    <xacro:property name="front_suspension_height" value="0.10669" />
     <xacro:property name="front_suspension_mass" value="${7850.0 * front_suspension_length * front_suspension_width * front_suspension_height}" />
     <!--Rear suspension dimensions -->
     <xacro:property name="rear_suspension_length" value="0.05" />
     <xacro:property name="rear_suspension_width" value="0.11" />
-    <xacro:property name="rear_suspension_height" value="0.105" />
+    <xacro:property name="rear_suspension_height" value="0.12169" />
     <xacro:property name="rear_suspension_mass" value="${7850.0 * rear_suspension_length * rear_suspension_width * rear_suspension_height}" />
     <!-- Wheel dimensions -->

File: traxxas_robot_description/urdf/zed2.xacro (robot description, xacro)
@@ -117,6 +117,6 @@
                 <horizontal_fov>1.3962634</horizontal_fov>
                 <image>
-                    <width>640</width>
-                    <height>480</height>
+                    <width>1920</width>
+                    <height>1024</height>
                     <format>R8G8B8</format>
                 </image>
@@ -147,6 +147,6 @@
                 <horizontal_fov>1.3962634</horizontal_fov>
                 <image>
-                    <width>640</width>
-                    <height>480</height>
+                    <width>1920</width>
+                    <height>1024</height>
                     <format>R8G8B8</format>
                 </image>
