Commit message: Updated robot simulation with PWM - Configured direction calculation using Ackermann model formula ω = V / L * tan(δ) - Updated launch file to execute PWM - cmd_vel node - Updated lidar position to match physical robot

File: traxxas_robot_description/urdf/lidar.xacro (robot description, xacro)
@@ -45,5 +45,5 @@
         <parent link="chassis_link" />
         <child link="lidar_base_link" />
-        <origin xyz="${-chassis_length/2 + lidar_base_length/2 + 0.025} 0 ${chassis_height + lidar_base_height/2}" rpy="0 0 0" />
+        <origin xyz="${-chassis_length/2 + lidar_base_length/2} 0 ${chassis_height + lidar_base_height/2}" rpy="0 0 0" />
         <axis xyz="0 1 0" />
     </joint>

File: traxxas_robot_description/urdf/mobile_base.xacro (robot description, xacro)
@@ -29,5 +29,5 @@
     <xacro:property name="max_steering_angular_vel" value="1.570796" />
     <xacro:property name="max_steering_effort" value="1.0" />
-    <xacro:property name="max_vel" value="15.665470085" />
+    <xacro:property name="max_vel" value="4" />
     <xacro:property name="max_effort" value="10.0" />
     <xacro:property name="max_wheel_angular_vel" value="${max_vel / wheel_radius}" />
